File: HG0B1CEU6N/Design/STM32-G0-Dip-Module.sch (EAGLE design)
At the start: 29 parts, among them U1 STM32G0B1CEU6NUFQFPN48_STM32_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, U2 TPS76433DBVT, X1 XTALL_CSTCE8M00G52

Commit message: -Changing the Schematic design stile -Correcting some BOM-file data
Other:
- note added: "0"
- note added: "1"
- note added: "Author"
- note added: "C:/Users/Admin/Desktop/logodraft.bmp"
- note added: "Description"
- note added: "HG0B1CEU6"
- note added: "Ibrahim Zaeiter"
- note added: "Letter"
- note added: "Revision"
- note added: "STM32G0B1CEU6N DevKit"
- note added: "Sheet of"
- note added: "Size"
- note added: "Title"
- note added: "www.hexabitz.com"
