File: HG0B1CEU6N_V2/Design/STM32-G0-Dip-Module.sch (EAGLE design)
At the start: 35 parts, among them U1 STM32G0B1CEU6QFN_B1CEU6_STM-L, U2 TPS76433DBVT, X1 XTALL_CSTCE8M00G52

Commit message: -Correcting some documentaion issues
Other:
- note added: "2"
Changed lines of the file:
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@@
 <?xml version="1.0" encoding="utf-8"?>
 <!DOCTYPE eagle SYSTEM "eagle.dtd">
-<eagle version="9.6.1">
+<eagle version="9.6.2">
 <drawing>
 <settings>
@@
 <text x="82.8802" y="-95.7834" size="1.9304" layer="101" font="vector">1</text>
 <text x="78.74" y="-105.1052" size="1.9304" layer="101" font="vector">1</text>
-<text x="83.566" y="-105.1052" size="1.9304" layer="101" font="vector">1</text>
+<text x="83.566" y="-105.1052" size="1.9304" layer="101" font="vector">2</text>
 <wire x1="86.36" y1="-106.68" x2="86.36" y2="-92.202" width="0.1524" layer="205"/>
 <wire x1="24.13" y1="-87.63" x2="86.36" y2="-87.63" width="0.1524" layer="205"/>
@@
 <text x="86.36" y="-92.6592" size="1.9304" layer="101" font="vector">Letter</text>
 <text x="91.7702" y="-88.1634" size="1.9304" layer="101" font="vector">1</text>
-<text x="87.63" y="-97.4852" size="1.9304" layer="101" font="vector">1</text>
-<text x="92.456" y="-97.4852" size="1.9304" layer="101" font="vector">1</text>
+<text x="87.63" y="-97.4852" size="1.9304" layer="101" font="vector">2</text>
+<text x="92.456" y="-97.4852" size="1.9304" layer="101" font="vector">2</text>
 <wire x1="95.25" y1="-99.06" x2="95.25" y2="-84.582" width="0.1524" layer="205"/>
 <wire x1="33.02" y1="-80.01" x2="95.25" y2="-80.01" width="0.1524" layer="205"/>
